File: ATtiny84LEDEL.brd (EAGLE design)
At the start: 69.9 x 25.4 mm, 28 parts, among them Q1 MOSFET-NCHANNELPTH, Q2 MOSFET-NCHANNELPTH, Q3 MOSFET-NCHANNELPTH, U1 ATTINY84-20PU, U2 MOC3043M, U3 BTA06

Commit message: Updated Eagle PCB files.
Parts:
- removed LED1, LED2, LED3: (no value), adafruit:LED5MM
- removed U$2: (no value), ohw-logo:OSHW_FILLX200_NOTEXT
- added 1, 2, 3: (no value), adafruit:LED5MM
- added U$1: (no value), ohw-logo:OSHW_FILLX150_NOTEXT
- moved R10 59.1 mm to (26.7, 17.8), turned to 180 degrees
- moved BAT1 36.4 mm to (19.1, 1.65), turned to 90 degrees
- moved R9 23.6 mm to (26.7, 20.3), turned to 180 degrees
- moved R8 19.4 mm to (26.7, 22.9), turned to 180 degrees
- moved R7 16.5 mm to (53.5, 15.2), turned to 270 degrees
- moved R2 12.9 mm to (14.0, 23.1)
- moved J1 12.2 mm to (72.8, 4.32)
- moved J2 12.2 mm to (72.8, 16.0)
- moved Q1 11.9 mm to (15.7, 18.8)
- moved Q3 7.16 mm to (15.7, 3.05), turned to 0 degrees
- moved Q2 6.41 mm to (15.7, 10.9), turned to 0 degrees
- moved R3 4.77 mm to (14.0, 15.2), turned to 180 degrees
- moved U3 4.66 mm to (63.1, 15.4), turned to 180 degrees
- moved R4 3.27 mm to (14.0, 7.37), turned to 180 degrees
- moved JP2 2.54 mm to (34.3, 22.9)
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Connections:
- removed net N$13: J2.1, R7.P$1, U3.1
- removed net N$17: J1.2, R6.P$1, U3.2
- removed net N$9: J1.1, J2.2
- new net AC1: J1.1, R6.P$1, U3.2
- new net AC2: J1.2, J2.1
- new net AC3: J2.2, R7.P$1, U3.1
- net D0: now also JP2.3; no longer JP2.5
- net D1: now also JP2.2; no longer JP2.4
- net D10/A0: now also JP2.4; no longer JP2.6
- net D7/A3: now also JP2.1; no longer JP2.3
- net GND: now also JP2.6; no longer JP2.1
- net N$12: now also 2.A; no longer LED2.A
- net N$14: now also 3.A; no longer LED3.A
- net N$3: now also 1.K; no longer LED1.K
- net N$4: now also 2.K; no longer LED2.K
- net N$6: now also 3.K; no longer LED3.K
- net N$8: now also 1.A; no longer LED1.A
- net VCC: now also JP2.5; no longer JP2.2
Routing:
- net N$17: track 24.0 -> 0.00 mm
- net VCC: track 77.2 -> 94.9 mm
- net N$7: track 16.4 -> 0.00 mm, vias 1 -> 0
- net N$13: track 10.0 -> 0.00 mm
- net D2: track 13.0 -> 22.3 mm
- net N$5: track 6.59 -> 0.00 mm
- net N$10: track 3.18 -> 0.00 mm, vias 1 -> 0
- net D4/MOSI: track 27.1 -> 24.1 mm
- net N$14: track 5.76 -> 3.11 mm
- net N$6: track 3.18 -> 5.25 mm
- net N$3: track 3.18 -> 5.25 mm
- net RST: track 28.4 -> 26.6 mm
- net N$12: track 4.87 -> 3.11 mm
- net N$4: track 3.60 -> 5.25 mm
- net N$8: track 4.45 -> 3.11 mm
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- added copper zone on layer 1, net AC1
- added copper zone on layer 16, net AC1
- added copper zone on layer 16, net AC2
- added copper zone on layer 1, net AC3
- added copper zone on layer 16, net AC3
- added copper zone on layer 16, net N$5
- added copper zone on layer 16, net N$7
Other:
- board text added: "HIGH"
- board text added: "VOLTAGE"
- board text removed: "HV"
- board text removed: "LV"
