File: ATtiny84LEDEL.sch (EAGLE design)
At the start: 27 parts, among them Q1 MOSFET-NCHANNELPTH, Q2 MOSFET-NCHANNELPTH, Q3 MOSFET-NCHANNELPTH, U1 ATTINY84-20PU, U2 MOC3043M, U3 BTA06

Commit message: Updated Eagle PCB files.
Parts:
- removed LED1, LED2, LED3: (no value), adafruit:LED5MM
- added 1, 2, 3: (no value), adafruit:LED5MM
Connections:
- removed net N$13: J2.1, R7.1, U3.A1
- removed net N$17: J1.2, R6.1, U3.A2
- removed net N$9: J1.1, J2.2
- new net AC1: J1.1, R6.1, U3.A2
- new net AC2: J1.2, J2.1
- new net AC3: J2.2, R7.1, U3.A1
- net D0: now also JP2.3; no longer JP2.5
- net D1: now also JP2.2; no longer JP2.4
- net D10/A0: now also JP2.4; no longer JP2.6
- net D7/A3: now also JP2.1; no longer JP2.3
- net GND: now also JP2.6; no longer JP2.1
- net N$12: now also 2.A; no longer LED2.A
- net N$14: now also 3.A; no longer LED3.A
- net N$3: now also 1.C; no longer LED1.C
- net N$4: now also 2.C; no longer LED2.C
- net N$6: now also 3.C; no longer LED3.C
- net N$8: now also 1.A; no longer LED1.A
- net VCC: now also JP2.5; no longer JP2.2
Other:
- note removed: "1 February 2013"
- note removed: "ATtiny84 LED + EL"
- note removed: "Version 1.0"
- note removed: "http://www.digitalmisery.com"
- moved on the sheet: BAT1, C1, C2, ISP1, JP1, JP2, Q1, Q2, Q3, R1, R10, R2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

Commit message: Added frame to schematic.
Other:
- note added: "6 February 2013"
- note added: "ATtiny84 LED + EL"
- note added: "Revision 1.1"
- note added: "http://www.digitalmisery.com"
- moved on the sheet: 1, 2, 3, BAT1, C1, C2, ISP1, JP1, JP2, Q1, Q2, Q3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
